Commit message: Modified meshes

File: urdf/bolt.gazebo.xacro (robot description, xacro)
@@ -13,4 +13,20 @@
         <material>Gazebo/Black</material>
     </gazebo>
+    <gazebo reference="rear_left_wheel">
+        <mu1>0.4</mu1>
+        <mu2>0.4</mu2>
+    </gazebo>
+    <gazebo reference="rear_right_wheel">
+        <mu1>0.4</mu1>
+        <mu2>0.4</mu2>
+    </gazebo>
+    <gazebo reference="front_left_wheel">
+        <mu1>0.4</mu1>
+        <mu2>0.4</mu2>
+    </gazebo>
+    <gazebo reference="front_right_wheel">
+        <mu1>0.4</mu1>
+        <mu2>0.4</mu2>
+    </gazebo>
     <!-- ROS Controller plugin -->
     <gazebo>

File: urdf/bolt.urdf.xacro (robot description, xacro)
@@ -81,7 +81,7 @@
         </collision>
         <visual>
-            <origin xyz="0 0 0" rpy="1.57075 0 0" />
-            <geometry>
-                <cylinder length="0.14" radius="0.2286" />
+            <origin xyz="0 0 0" rpy="0 0 0" />
+            <geometry>
+                <mesh filename="package://igvc_bolt/meshes/Wheel.dae" scale="1.8 1.8 1.8" />
             </geometry>
         </visual>
@@ -106,7 +106,7 @@
         </collision>
         <visual>
-            <origin xyz="0 0 0" rpy="1.57075 0 0" />
-            <geometry>
-                <cylinder length="0.14" radius="0.2286" />
+            <origin xyz="0 0 0" rpy="0 0 0" />
+            <geometry>
+                <mesh filename="package://igvc_bolt/meshes/Wheel.dae" scale="1.8 1.8 1.8" />
             </geometry>
         </visual>
@@ -226,7 +226,7 @@
         </collision>
         <visual>
-            <origin xyz="0 0 0" rpy="1.57075 0 0" />
-            <geometry>
-                <cylinder length="0.14" radius="0.2286" />
+            <origin xyz="0 0 0" rpy="0 0 0" />
+            <geometry>
+                <mesh filename="package://igvc_bolt/meshes/Wheel.dae" scale="1.8 1.8 1.8" />
             </geometry>
         </visual>
@@ -299,7 +299,7 @@
         </collision>
         <visual>
-            <origin xyz="0 0 0" rpy="1.57075 0 0" />
-            <geometry>
-                <cylinder length="0.14" radius="0.2286" />
+            <origin xyz="0 0 0" rpy="0 0 0" />
+            <geometry>
+                <mesh filename="package://igvc_bolt/meshes/Wheel.dae" scale="1.8 1.8 1.8" />
             </geometry>
         </visual>

Commit message: Added sensors

File: urdf/bolt.gazebo.xacro (robot description, xacro)
@@ -1,4 +1,4 @@
 <?xml version="1.0"?>
-<robot name="final" xmlns:xacro="http://www.ros.org/wiki/xacro">
+<robot name="bolt" xmlns:xacro="http://www.ros.org/wiki/xacro">
     <gazebo reference="front_left_wheel">
         <material>Gazebo/Black</material>
@@ -37,3 +37,225 @@
         </plugin>
     </gazebo>
+    <!-- Cameras -->
+    <gazebo reference="camera_front_left">
+        <sensor type="camera" name="camera_front_left">
+            <update_rate>30.0</update_rate>
+            <camera name="camera_front_left">
+                <horizontal_fov>2</horizontal_fov>
+                <image>
+                    <width>800</width>
+                    <height>800</height>
+                    <format>R8G8B8</format>
+                </image>
+                <clip>
+                    <near>0.02</near>
+                    <far>300</far>
+                </clip>
+                <noise>
+                    <type>gaussian</type>
+                    <mean>0.0</mean>
+                    <stddev>0.007</stddev>
+                </noise>
+            </camera>
+            <plugin name="camera_controller" filename="libgazebo_ros_camera.so">
+                <robotNamespace>/</robotNamespace>
+                <alwaysOn>true</alwaysOn>
+                <updateRate>0.0</updateRate>
+                <cameraName>camera/front/left</cameraName>
+                <imageTopicName>image_raw</imageTopicName>
+                <cameraInfoTopicName>camera_info</cameraInfoTopicName>
+                <frameName>camera_front_left</frameName>
+                <hackBaseline>0.07</hackBaseline>
+                <distortionK1>0.0</distortionK1>
+                <distortionK2>0.0</distortionK2>
+                <distortionK3>0.0</distortionK3>
+                <distortionT1>0.0</distortionT1>
+                <distortionT2>0.0</distortionT2>
+            </plugin>
+        </sensor>
+    </gazebo>
+    <gazebo reference="camera_front_right">
+        <sensor type="camera" name="camera_front_right">
+            <update_rate>30.0</update_rate>
+            <camera name="camera_front_right">
+                <horizontal_fov>2</horizontal_fov>
+                <image>
+                    <width>800</width>
+                    <height>800</height>
+                    <format>R8G8B8</format>
+                </image>
+                <clip>
+                    <near>0.02</near>
+                    <far>300</far>
+                </clip>
+                <noise>
+                    <type>gaussian</type>
+                    <mean>0.0</mean>
+                    <stddev>0.007</stddev>
+                </noise>
+            </camera>
+            <plugin name="camera_controller" filename="libgazebo_ros_camera.so">
+                <robotNamespace>/</robotNamespace>
+                <alwaysOn>true</alwaysOn>
+                <updateRate>0.0</updateRate>
+                <cameraName>camera/front/right</cameraName>
+                <imageTopicName>image_raw</imageTopicName>
+                <cameraInfoTopicName>camera_info</cameraInfoTopicName>
+                <frameName>camera_front_right</frameName>
+                <hackBaseline>0.07</hackBaseline>
+                <distortionK1>0.0</distortionK1>
+                <distortionK2>0.0</distortionK2>
+                <distortionK3>0.0</distortionK3>
+                <distortionT1>0.0</distortionT1>
+                <distortionT2>0.0</distortionT2>
+            </plugin>
+        </sensor>
+    </gazebo>
+    <gazebo reference="camera_rear_left">
+        <sensor type="camera" name="camera_rear_left">
+            <update_rate>30.0</update_rate>
+            <camera name="camera_rear_left">
+                <horizontal_fov>2</horizontal_fov>
+                <image>
+                    <width>800</width>
+                    <height>800</height>
+                    <format>R8G8B8</format>
+                </image>
+                <clip>
+                    <near>0.02</near>
+                    <far>300</far>
+                </clip>
+                <noise>
+                    <type>gaussian</type>
+                    <mean>0.0</mean>
+                    <stddev>0.007</stddev>
+                </noise>
+            </camera>
+            <plugin name="camera_controller" filename="libgazebo_ros_camera.so">
+                <robotNamespace>/</robotNamespace>
+                <alwaysOn>true</alwaysOn>
+                <updateRate>0.0</updateRate>
+                <cameraName>camera/rear/left</cameraName>
+                <imageTopicName>image_raw</imageTopicName>
+                <cameraInfoTopicName>camera_info</cameraInfoTopicName>
+                <frameName>camera_rear_left</frameName>
+                <hackBaseline>0.07</hackBaseline>
+                <distortionK1>0.0</distortionK1>
+                <distortionK2>0.0</distortionK2>
+                <distortionK3>0.0</distortionK3>
+                <distortionT1>0.0</distortionT1>
+                <distortionT2>0.0</distortionT2>
+            </plugin>
+        </sensor>
+    </gazebo>
+    <gazebo reference="camera_rear_right">
+        <sensor type="camera" name="camera_rear_right">
+            <update_rate>30.0</update_rate>
+            <camera name="camera_rear_right">
+                <horizontal_fov>2</horizontal_fov>
+                <image>
+                    <width>800</width>
+                    <height>800</height>
+                    <format>R8G8B8</format>
+                </image>
+                <clip>
+                    <near>0.02</near>
+                    <far>300</far>
+                </clip>
+                <noise>
+                    <type>gaussian</type>
+                    <mean>0.0</mean>
+                    <stddev>0.007</stddev>
+                </noise>
+            </camera>
+            <plugin name="camera_controller" filename="libgazebo_ros_camera.so">
+                <robotNamespace>/</robotNamespace>
+                <alwaysOn>true</alwaysOn>
+                <updateRate>0.0</updateRate>
+                <cameraName>camera/rear/right</cameraName>
+                <imageTopicName>image_raw</imageTopicName>
+                <cameraInfoTopicName>camera_info</cameraInfoTopicName>
+                <frameName>camera_rear_right</frameName>
+                <hackBaseline>0.07</hackBaseline>
+                <distortionK1>0.0</distortionK1>
+                <distortionK2>0.0</distortionK2>
+                <distortionK3>0.0</distortionK3>
+                <distortionT1>0.0</distortionT1>
+                <distortionT2>0.0</distortionT2>
+            </plugin>
+        </sensor>
+    </gazebo>
+    <!-- Laser -->
+    <gazebo reference="laser">
+        <material>Gazebo/Grey</material>
+        <sensor type="ray" name="lds_lfcd_sensor">
+            <pose>0 0 0 0 0 0</pose>
+            <visualize>true</visualize>
+            <update_rate>20</update_rate>
+            <ray>
+                <scan>
+                    <horizontal>
+                        <samples>360</samples>
+                        <resolution>1</resolution>
+                        <min_angle>-1.57</min_angle>
+                        <max_angle>1.57</max_angle>
+                    </horizontal>
+                </scan>
+                <range>
+                    <min>0.1</min>
+                    <max>12</max>
+                    <resolution>0.015</resolution>
+                </range>
+                <noise>
+                    <type>gaussian</type>
+                    <mean>0.0</mean>
+                    <stddev>0.01</stddev>
+                </noise>
+            </ray>
+            <plugin name="gazebo_ros_lds_lfcd_controller" filename="libgazebo_ros_laser.so">
+                <robotNamespace>/</robotNamespace>
+                <topicName>/laser/scan</topicName>
+                <frameName>laser</frameName>
+            </plugin>
+        </sensor>
+    </gazebo>
+    <!-- IMU -->
+    <gazebo reference="imu">
+        <material>Gazebo/Grey</material>
+        <gravity>true</gravity>
+        <sensor name="imu_sensor" type="imu">
+            <always_on>true</always_on>
+            <update_rate>100</update_rate>
+            <visualize>true</visualize>
+            <topic>__default_topic__</topic>
+            <plugin filename="libgazebo_ros_imu_sensor.so" name="imu_plugin">
+                <robotNamespace>/</robotNamespace>
+                <topicName>imu</topicName>
+                <bodyName>imu</bodyName>
+                <updateRateHZ>10.0</updateRateHZ>
+                <gaussianNoise>0.0</gaussianNoise>
+                <xyzOffset>0 0 0</xyzOffset>
+                <rpyOffset>0 0 0</rpyOffset>
+                <frameName>imu</frameName>
+                <initialOrientationAsReference>false</initialOrientationAsReference>
+            </plugin>
+            <pose>0 0 0 0 0 0</pose>
+        </sensor>
+    </gazebo>
+    <!-- GPS -->
+    <gazebo reference="gps">
+        <plugin name="gps" filename="libhector_gazebo_ros_gps.so">
+            <robotNamespace>/</robotNamespace>
+            <alwaysOn>1</alwaysOn>
+            <updateRate>10.0</updateRate>
+            <bodyName>gps</bodyName>
+            <frameId>gps</frameId>
+            <topicName>fix</topicName>
+            <velocityTopicName>fix_velocity</velocityTopicName>
+            <drift>5.0 5.0 5.0</drift>
+            <gaussianNoise>0.1 0.1 0.1</gaussianNoise>
+            <velocityDrift>0 0 0</velocityDrift>
+            <velocityGaussianNoise>0.1 0.1 0.1</velocityGaussianNoise>
+        </plugin>
+    </gazebo>
 </robot>

File: urdf/bolt.urdf.xacro (robot description, xacro)
@@ -1,5 +1,6 @@
 <?xml version="1.0"?>
-<robot name="virat" xmlns:xacro="http://www.ros.org/wiki/xacro">
+<robot name="bolt" xmlns:xacro="http://www.ros.org/wiki/xacro">
     <xacro:include filename="$(find igvc_bolt)/urdf/bolt.gazebo.xacro" />
+    <xacro:include filename="$(find igvc_bolt)/urdf/bolt.trans.xacro" />
     <xacro:include filename="$(find igvc_bolt)/urdf/materials.xacro" />
     <link name="base_link"></link>
@@ -32,5 +33,5 @@
     <!-- Rear wheel - Bicycle model -->
     <link name="rear_wheel">
-        <inertial>
+        <!-- <inertial>
             <mass value="1" />
             <origin xyz="0 0 0" rpy="0 0 0" />
@@ -42,5 +43,5 @@
                 <cylinder length="0.1" radius="0.08" />
             </geometry>
-        </collision>
+        </collision> -->
         <visual>
             <origin xyz="0 0 0" rpy="1.57075 0 0" />
@@ -50,20 +51,4 @@
         </visual>
     </link>
-    <joint name="rear_wheel_joint" type="continuous">
-        <axis xyz="0 1 0" />
-        <parent link="chassis" />
-        <child link="rear_wheel" />
-        <origin xyz="-1.0 0 0.01" rpy="0 0 0" />
-    </joint>
-    <transmission name="rear_wheel_joint_trans">
-        <type>transmission_interface/SimpleTransmission</type>
-        <actuator name="rear_wheel_joint_motor">
-            <mechanicalReduction>1</mechanicalReduction>
-            <hardwareInterface>hardware_interface/VelocityJointInterface</hardwareInterface>
-        </actuator>
-        <joint name="rear_wheel_joint">
-            <hardwareInterface>hardware_interface/VelocityJointInterface</hardwareInterface>
-        </joint>
-    </transmission>
     <!-- *************************************************************************************************** -->
     <!-- Rear wheels (Left & Right) - Steering Model -->
@@ -118,24 +103,4 @@
         <origin xyz="-1.05 -0.7 0.01" rpy="0 0 0" />
     </joint>
-    <transmission name="rear_right_wheel_joint_trans">
-        <type>transmission_interface/SimpleTransmission</type>
-        <joint name="rear_right_wheel_joint">
-            <hardwareInterface>hardware_interface/VelocityJointInterface</hardwareInterface>
-        </joint>
-        <actuator name="rear_right_wheel_motor">
-            <hardwareInterface>hardware_interface/VelocityJointInterface</hardwareInterface>
-            <mechanicalReduction>1</mechanicalReduction>
-        </actuator>
-    </transmission>
-    <transmission name="rear_left_wheel_joint_trans">
-        <type>transmission_interface/SimpleTransmission</type>
-        <joint name="rear_left_wheel_joint">
-            <hardwareInterface>hardware_interface/VelocityJointInterface</hardwareInterface>
-        </joint>
-        <actuator name="rear_left_wheel_motor">
-            <hardwareInterface>hardware_interface/VelocityJointInterface</hardwareInterface>
-            <mechanicalReduction>1</mechanicalReduction>
-        </actuator>
-    </transmission>
     <!-- ********************************************************************************************* -->
     <!-- Front steer - Bicycle Model -->
@@ -166,14 +131,4 @@
         <limit effort="7.0" velocity="${200.0*3.1415/180.0*0.95}" />
     </joint>
-    <transmission name="front_steer_joint_trans">
-        <type>transmission_interface/SimpleTransmission</type>
-        <actuator name="front_steer_joint_motor">
-            <mechanicalReduction>1</mechanicalReduction>
-            <hardwareInterface>hardware_interface/PositionJointInterface</hardwareInterface>
-        </actuator>
-        <joint name="front_steer_joint">
-            <hardwareInterface>hardware_interface/PositionJointInterface</hardwareInterface>
-        </joint>
-    </transmission>
     <!-- ************************************************************************************* -->
     <!-- Front left steer and wheel links-->
@@ -203,14 +158,4 @@
         <limit effort="7.0" velocity="${200.0*3.1415/180.0*0.95}" />
     </joint>
-    <transmission name="front_left_steer_joint_trans">
-        <type>transmission_interface/SimpleTransmission</type>
-        <actuator name="front_left_steer_joint_motor">
-            <mechanicalReduction>1</mechanicalReduction>
-            <hardwareInterface>hardware_interface/PositionJointInterface</hardwareInterface>
-        </actuator>
-        <joint name="front_left_steer_joint">
-            <hardwareInterface>hardware_interface/PositionJointInterface</hardwareInterface>
-        </joint>
-    </transmission>
     <link name="front_left_wheel">
         <inertial>
@@ -238,14 +183,4 @@
         <origin xyz="0 0 -0.29" rpy="0 0 0" />
     </joint>
-    <transmission name="front_left_wheel_joint_trans">
-        <type>transmission_interface/SimpleTransmission</type>
-        <joint name="front_left_wheel_joint">
-            <hardwareInterface>hardware_interface/VelocityJointInterface</hardwareInterface>
-        </joint>
-        <actuator name="front_left_wheel_motor">
-            <hardwareInterface>hardware_interface/VelocityJointInterface</hardwareInterface>
-            <mechanicalReduction>1</mechanicalReduction>
-        </actuator>
-    </transmission>
     <!-- **************************************************************************************** -->
     <!-- Front right steer and wheel links -->
@@ -274,16 +209,6 @@
         <child link="front_right_steer" />
         <origin xyz="0.85 -0.7 0.3" rpy="0 0 0" />
-        <limit effort="7.0"  velocity="${200.0*3.1415/180.0*0.95}" />
-    </joint>
-    <transmission name="front_right_steer_joint_trans">
-        <type>transmission_interface/SimpleTransmission</type>
-        <actuator name="front_right_steer_joint_motor">
-            <mechanicalReduction>1</mechanicalReduction>
-            <hardwareInterface>hardware_interface/PositionJointInterface</hardwareInterface>
-        </actuator>
-        <joint name="front_right_steer_joint">
-            <hardwareInterface>hardware_interface/PositionJointInterface</hardwareInterface>
-        </joint>
-    </transmission>
+        <limit effort="7.0" velocity="${200.0*3.1415/180.0*0.95}" />
+    </joint>
     <link name="front_right_wheel">
         <inertial>
@@ -311,14 +236,93 @@
         <origin xyz="0 0 -0.29" rpy="0 0 0" />
     </joint>
-    <transmission name="front_right_wheel_joint_trans">
-        <type>transmission_interface/SimpleTransmission</type>
-        <joint name="front_right_wheel_joint">
-            <hardwareInterface>hardware_interface/VelocityJointInterface</hardwareInterface>
-        </joint>
-        <actuator name="front_right_wheel_motor">
-            <hardwareInterface>hardware_interface/VelocityJointInterface</hardwareInterface>
-            <mechanicalReduction>1</mechanicalReduction>
-        </actuator>
-    </transmission>
     <!-- ************************************************************************************************************* -->
+    <!-- CAMERAS - 4 -->
+    <link name="camera_front_left">
+        <visual>
+            <origin xyz="0 0 0" rpy="0 0 0" />
+            <geometry>
+                <cylinder radius="0.01" length="0.005" />
+            </geometry>
+        </visual>
+    </link>
+    <joint name="camera_front_left_joint" type="fixed">
+        <parent link="chassis" />
+        <child link="camera_front_left" />
+        <origin xyz="1.05 0.6 0.55" rpy="0 0 0.15" />
+    </joint>
+    <link name="camera_front_right">
+        <visual>
+            <origin xyz="0 0 0" rpy="0 0 0" />
+            <geometry>
+                <cylinder radius="0.01" length="0.005" />
+            </geometry>
+        </visual>
+    </link>
+    <joint name="camera_front_right_joint" type="fixed">
+        <parent link="chassis" />
+        <child link="camera_front_right" />
+        <origin xyz="1.05 -0.6 0.55" rpy="0 0 -0.15" />
+    </joint>
+    <link name="camera_rear_left">
+        <visual>
+            <origin xyz="0 0 0" rpy="0 0 0" />
+            <geometry>
+                <cylinder radius="0.01" length="0.005" />
+            </geometry>
+        </visual>
+    </link>
+    <joint name="camera_rear_left_joint" type="fixed">
+        <parent link="chassis" />
+        <child link="camera_rear_left" />
+        <origin xyz="-0.85 0.6 0.6" rpy="0 0 2.991" />
+    </joint>
+    <link name="camera_rear_right">
+        <visual>
+            <origin xyz="0 0 0" rpy="0 0 0" />
+            <geometry>
+                <cylinder radius="0.01" length="0.005" />
+            </geometry>
+        </visual>
+    </link>
+    <joint name="camera_rear_right_joint" type="fixed">
+        <parent link="chassis" />
+        <child link="camera_rear_right" />
+        <origin xyz="-0.85 -0.6 0.6" rpy="0 0 -2.991" />
+    </joint>
+    <!-- ************************************************************************* -->
+    <!-- Laser -->
+    <link name="laser">
+        <visual>
+            <origin rpy="0 0 0" xyz="0 0 0" />
+            <geometry>
+                <mesh filename="package://igvc_bolt/meshes/Laser.dae" />
+            </geometry>
+        </visual>
+    </link>
+    <joint name="laser_joint" type="fixed">
+        <parent link="chassis" />
+        <child link="laser" />
+        <origin xyz="1 0.0 0.6" rpy="0.0 0.0 0.0" />
+    </joint>
+    <!-- IMU -->
+    <link name="imu">
+        <visual>
+            <origin xyz="0 0 0" rpy="0 0 0" />
+            <geometry>
+                <box size="0.2 0.1 0.01" />
+            </geometry>
+        </visual>
+    </link>
+    <joint name="imu_joint" type="fixed">
+        <parent link="chassis" />
+        <child link="imu" />
+        <origin xyz="0 0.0 1.48" rpy="0.0 0.0 0.0" />
+    </joint>
+    <!-- GPS -->
+    <link name="gps"></link>
+    <joint name="gps_joint" type="fixed">
+        <parent link="chassis" />
+        <child link="gps" />
+        <origin xyz="0.0 0.0 0.0" rpy="0.0 0.0 0.0" />
+    </joint>
 </robot>
