Commit message: teleop

File: urdf/bolt.gazebo.xacro (robot description, xacro)
@@ -44,5 +44,5 @@
                 <horizontal_fov>2</horizontal_fov>
                 <image>
-                    <width>800</width>
+                    <width>1200</width>
                     <height>800</height>
                     <format>R8G8B8</format>
@@ -81,5 +81,5 @@
                 <horizontal_fov>2</horizontal_fov>
                 <image>
-                    <width>800</width>
+                    <width>1200</width>
                     <height>800</height>
                     <format>R8G8B8</format>

File: urdf/bolt.urdf.xacro (robot description, xacro)
@@ -33,15 +33,4 @@
     <!-- Rear wheel - Bicycle model -->
     <link name="rear_wheel">
-        <!-- <inertial>
-            <mass value="1" />
-            <origin xyz="0 0 0" rpy="0 0 0" />
-            <inertia ixx="0.002433" ixy="0" ixz="0" iyy="0.0032" iyz="0" izz="0.002433" />
-        </inertial>
-        <collision>
-            <origin xyz="0 0 0" rpy="1.57075 0 0" />
-            <geometry>
-                <cylinder length="0.1" radius="0.08" />
-            </geometry>
-        </collision> -->
         <visual>
             <origin xyz="0 0 0" rpy="1.57075 0 0" />

Commit message: Remove two front cameras

File: urdf/bolt.gazebo.xacro (robot description, xacro)
@@ -38,8 +38,8 @@
     </gazebo>
     <!-- Cameras -->
-    <gazebo reference="camera_front_left">
-        <sensor type="camera" name="camera_front_left">
+    <gazebo reference="camera_front">
+        <sensor type="camera" name="camera_front">
             <update_rate>30.0</update_rate>
-            <camera name="camera_front_left">
+            <camera name="camera_front">
                 <horizontal_fov>2</horizontal_fov>
                 <image>
@@ -62,119 +62,8 @@
                 <alwaysOn>true</alwaysOn>
                 <updateRate>0.0</updateRate>
-                <cameraName>camera/front/left</cameraName>
+                <cameraName>camera/front</cameraName>
                 <imageTopicName>image_raw</imageTopicName>
                 <cameraInfoTopicName>camera_info</cameraInfoTopicName>
-                <frameName>camera_front_left</frameName>
-                <hackBaseline>0.07</hackBaseline>
-                <distortionK1>0.0</distortionK1>
-                <distortionK2>0.0</distortionK2>
-                <distortionK3>0.0</distortionK3>
-                <distortionT1>0.0</distortionT1>
-                <distortionT2>0.0</distortionT2>
-            </plugin>
-        </sensor>
-    </gazebo>
-    <gazebo reference="camera_front_right">
-        <sensor type="camera" name="camera_front_right">
-            <update_rate>30.0</update_rate>
-            <camera name="camera_front_right">
-                <horizontal_fov>2</horizontal_fov>
-                <image>
-                    <width>1920</width>
-                    <height>1080</height>
-                    <format>R8G8B8</format>
-                </image>
-                <clip>
-                    <near>0.02</near>
-                    <far>300</far>
-                </clip>
-                <noise>
-                    <type>gaussian</type>
-                    <mean>0.0</mean>
-                    <stddev>0.007</stddev>
-                </noise>
-            </camera>
-            <plugin name="camera_controller" filename="libgazebo_ros_camera.so">
-                <robotNamespace>/</robotNamespace>
-                <alwaysOn>true</alwaysOn>
-                <updateRate>0.0</updateRate>
-                <cameraName>camera/front/right</cameraName>
-                <imageTopicName>image_raw</imageTopicName>
-                <cameraInfoTopicName>camera_info</cameraInfoTopicName>
-                <frameName>camera_front_right</frameName>
-                <hackBaseline>0.07</hackBaseline>
-                <distortionK1>0.0</distortionK1>
-                <distortionK2>0.0</distortionK2>
-                <distortionK3>0.0</distortionK3>
-                <distortionT1>0.0</distortionT1>
-                <distortionT2>0.0</distortionT2>
-            </plugin>
-        </sensor>
-    </gazebo>
-    <gazebo reference="camera_rear_left">
-        <sensor type="camera" name="camera_rear_left">
-            <update_rate>30.0</update_rate>
-            <camera name="camera_rear_left">
-                <horizontal_fov>2</horizontal_fov>
-                <image>
-                    <width>800</width>
-                    <height>800</height>
-                    <format>R8G8B8</format>
-                </image>
-                <clip>
-                    <near>0.02</near>
-                    <far>300</far>
-                </clip>
-                <noise>
-                    <type>gaussian</type>
-                    <mean>0.0</mean>
-                    <stddev>0.007</stddev>
-                </noise>
-            </camera>
-            <plugin name="camera_controller" filename="libgazebo_ros_camera.so">
-                <robotNamespace>/</robotNamespace>
-                <alwaysOn>true</alwaysOn>
-                <updateRate>0.0</updateRate>
-                <cameraName>camera/rear/left</cameraName>
-                <imageTopicName>image_raw</imageTopicName>
-                <cameraInfoTopicName>camera_info</cameraInfoTopicName>
-                <frameName>camera_rear_left</frameName>
-                <hackBaseline>0.07</hackBaseline>
-                <distortionK1>0.0</distortionK1>
-                <distortionK2>0.0</distortionK2>
-                <distortionK3>0.0</distortionK3>
-                <distortionT1>0.0</distortionT1>
-                <distortionT2>0.0</distortionT2>
-            </plugin>
-        </sensor>
-    </gazebo>
-    <gazebo reference="camera_rear_right">
-        <sensor type="camera" name="camera_rear_right">
-            <update_rate>30.0</update_rate>
-            <camera name="camera_rear_right">
-                <horizontal_fov>2</horizontal_fov>
-                <image>
-                    <width>800</width>
-                    <height>800</height>
-                    <format>R8G8B8</format>
-                </image>
-                <clip>
-                    <near>0.02</near>
-                    <far>300</far>
-                </clip>
-                <noise>
-                    <type>gaussian</type>
-                    <mean>0.0</mean>
-                    <stddev>0.007</stddev>
-                </noise>
-            </camera>
-            <plugin name="camera_controller" filename="libgazebo_ros_camera.so">
-                <robotNamespace>/</robotNamespace>
-                <alwaysOn>true</alwaysOn>
-                <updateRate>0.0</updateRate>
-                <cameraName>camera/rear/right</cameraName>
-                <imageTopicName>image_raw</imageTopicName>
-                <cameraInfoTopicName>camera_info</cameraInfoTopicName>
-                <frameName>camera_rear_right</frameName>
+                <frameName>camera_front</frameName>
                 <hackBaseline>0.07</hackBaseline>
                 <distortionK1>0.0</distortionK1>

File: urdf/bolt.urdf.xacro (robot description, xacro)
@@ -227,5 +227,18 @@
     <!-- ************************************************************************************************************* -->
     <!-- CAMERAS - 4 -->
-    <link name="camera_front_left">
+    <link name="camera_front">
+        <visual>
+            <origin xyz="0 0 0" rpy="0 0 0"/>
+            <geometry>
+                <cylinder radius="0.01" length="0.005" />
+            </geometry>
+        </visual>
+    </link>
+    <joint name="camera_front_joint" type="fixed">
+        <parent link="chassis" />
+        <child link="camera_front" />
+        <origin xyz="1.05 0 0.55" rpy="0 0 0.15" />
+    </joint>
+    <!-- <link name="camera_front_left">
         <visual>
             <origin xyz="0 0 0" rpy="0 0 0" />
@@ -278,5 +291,5 @@
         <child link="camera_rear_right" />
         <origin xyz="-0.85 -0.6 0.6" rpy="0 0 -2.991" />
-    </joint>
+    </joint> -->
     <!-- ************************************************************************* -->
     <!-- Laser -->
