Commit message: Align camera properly

File: urdf/bolt.urdf.xacro (robot description, xacro)
@@ -238,5 +238,5 @@
         <parent link="chassis" />
         <child link="camera_front" />
-        <origin xyz="1.05 0 0.55" rpy="0 0 0.15" />
+        <origin xyz="1.05 0 0.55" rpy="0 0 0" />
     </joint>
     <!-- <link name="camera_front_left">
